File: cape.sch (EAGLE design)
At the start: 30 parts

Commit message: fix BB names int pinout
in the library adafruit
Parts:
- removed JP2: (no value), adafruit:PINHD-1X6B
- removed U$18: PINHD-1X10, adafruit:PINHD-1X10
- removed U$22, U$23: MOUNTINGHOLE3.0THIN, microbuilder:MOUNTINGHOLE3.0THIN
- added 12V_RELAYS: PINHD-1X10, adafruit:PINHD-1X10
- added AC_RELAYS: (no value), adafruit:PINHD-1X6B
- added FRAME1: FRAME-LEDGER, SparkFun-Aesthetics:FRAME-LEDGER
Connections:
- net GPIO_117 renamed LEVEL_MED
- net GPIO_50 renamed LEVEL_MAX
- net GPIO_51 renamed LEVEL_CW
- removed net GIPO_30: JP2.5
- removed net GPIO_20: U$18.6
- removed net GPIO_31: JP2.4
- removed net GPIO_48: U$18.5
- removed net GPIO_49: U$18.4
- removed net GPIO_67: U$18.8
- removed net GPIO_68: U$18.7
- removed net GPIO_69: U$18.9
- new net FAN: AC_RELAYS.2
- new net LEDS: AC_RELAYS.3
- new net LEVEL_MIN: LEVEL_MIN.1, R1.2
- new net N$1: U$2.GPIO_69
- new net NUT1: 12V_RELAYS.3
- new net NUT2: 12V_RELAYS.4
- new net NUT3: 12V_RELAYS.5
- new net PH+: 12V_RELAYS.6
- new net PH-: 12V_RELAYS.7
- new net WATER: 12V_RELAYS.2
- net GND: now also 12V_RELAYS.1, AC_RELAYS.1; no longer JP2.1, U$18.1
- net GPIO_115: now also U$2.GPIO_47; no longer LEVEL_MIN.1, R1.2, U$2.GPIO1_15
- net VCC: now also 12V_RELAYS.10, AC_RELAYS.6; no longer JP2.6, U$18.10
Other:
- note added: "LIGHT_SENSOR/ON-OFF/MUSIC/GPIO"
- note added: "POWER SUPPLY"
- moved on the sheet: DHT22, DS18B20, LEVEL_CW, LEVEL_CW1, LEVEL_MAX, LEVEL_MAX1, LEVEL_MED, LEVEL_MIN, R1, R11, R12, R2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

Commit message: change conectors to smd
and add 4 relays
Parts:
- removed 5V_IN: JST-PH_2-PIN_HEADER, SRG:JST-PH_2-PIN_HEADER
- removed DHT22, I2C_EC, I2C_PH, LEVEL_CW1, LEVEL_MAX1, LEVEL_MED, LEVEL_MED1, LEVEL_MIN1: JST-PH_4-PIN_HEADER, SRG:JST-PH_4-PIN_HEADER
- added +5V: BM02B-SRSS-TB, con-jst:BM02B-SRSS-TB
- added DHT, EC, GPIO, LDR, LEVE_MED, MUSIC, ON/OFF, PH: BM04B-SRSS-TB, con-jst:BM04B-SRSS-TB
- added Q1: MOSFET-NCHANNELBSS123LT1G, SparkFun-DiscreteSemi:MOSFET-NCHANNELBSS123LT1G
- added R13: 4.7K, adafruit:R-US_R0805
- added R14, R15: 10K, adafruit:R-US_R0805
- added U$1, U$3: FIDUCIAL, adafruit:FIDUCIAL
- DS18B20, LEVEL_CW, LEVEL_MAX, LEVEL_MIN: value JST-PH_4-PIN_HEADER -> BM04B-SRSS-TB; device SRG:JST-PH_4-PIN_HEADER -> con-jst:BM04B-SRSS-TB
- R1, R10, R11, R12, R2, R3, R4, R9: value (none) -> 10K
- R5, R6, R8: value 4k7 -> 4.7K
- R7: value 4k7 -> 100
Connections:
- removed net GPIO_115: U$2.GPIO_47
- new net 12V_1: 12V_RELAYS.8, U$2.GPIO_117
- new net 12V_2: 12V_RELAYS.9, U$2.ECAPPWM0
- new net AC_1: AC_RELAYS.4, U$2.EHRPWM1A
- new net AC_2: AC_RELAYS.5, U$2.GPIO_115
- new net LEVE_CW: LEVEL_CW-4.S
- new net N1: DS18B20-1.S, R13.1, R7.1
- new net VDD_3V3: DS18B20-4.S, EC-4.S, GPIO-4.S, LDR-4.S, MUSIC-4.S, ON/OFF-4.S, PH-4.S, R1.1, R10.1, R11.1, R12.1, R13.2, R15.2, R2.1, R3.1, R4.1, R5.2, R6.2, R9.1, U$2.VDD_3V3EXP@1, U$2.VDD_3V3EXP@2
- net DHT_AM2302: now also Q1.S, R15.1, U$2.SPI0_SCLK; no longer DHT22.3
- net DIGITAL_LDR: now also LDR-1.S, U$2.GPIO_66; no longer LEVEL_MIN1.1
- net DS18B20: now also R7.2, U$2.SPI0_D0; no longer DS18B20.3
- net FAN: now also U$2.UART4_TXD
- net GND: now also +5V-1.S, DHT-3.S, DS18B20-3.S, EC-3.S, GPIO-3.S, LDR-3.S, LEVEL_MAX-4.S, LEVEL_MIN-4.S, LEVE_MED-4.S, MUSIC-3.S, ON/OFF-3.S, PH-3.S, U$2.GND@1, U$2.GND@2, U$2.GND@7, U$2.GND@8; no longer 5V_IN.2, DHT22.1, DS18B20.1, I2C_EC.2, I2C_PH.2, R1.1, R10.1, R11.1, R12.1, R2.1, R3.1, R4.1, R9.1
- net GPIO: now also GPIO-1.S, U$2.LCD_VSYNC; no longer LEVEL_CW1.1
- net LEDS: now also U$2.UART4_RXD
- net LEVEL_CW: now also LEVEL_CW-1.S, U$2.LCD_DATA13; no longer LEVEL_CW.1
- net LEVEL_MAX: now also LEVEL_MAX-1.S, U$2.LCD_AC_BIAS; no longer LEVEL_MAX.1
- net LEVEL_MED: now also LEVE_MED-1.S, U$2.LCD_DATA11; no longer LEVEL_MED.1
- net LEVEL_MIN: now also LEVEL_MIN-1.S, U$2.LCD_DATA15; no longer LEVEL_MIN.1
- net MUSIC: now also MUSIC-1.S, U$2.EHRPWM2A; no longer LEVEL_MAX1.1
- net N$1: now also DHT-1.S, Q1.D, R14.1, R8.1; no longer U$2.GPIO_69
- net NUT1: now also U$2.GPIO_67
- net NUT2: now also U$2.GPIO_68
- net NUT3: now also U$2.GPIO_20
- net ON/OFF: now also ON/OFF-1.S, U$2.EHRPWM2B; no longer LEVEL_MED1.1
- net PH+: now also U$2.GPIO_48
- net PH-: now also U$2.UART1_TXD
- net SCL: now also EC-1.S, PH-1.S, R6.1; no longer I2C_EC.4, I2C_PH.4, R5.1, R7.1
- net SDA: now also EC-2.S, PH-2.S, R5.1; no longer I2C_EC.3, I2C_PH.3, R6.1, R8.1
- net VCC: now also +5V-2.S, DHT-4.S, Q1.G, R14.2; no longer 5V_IN.1, DHT22.4, DS18B20.4, I2C_EC.1, I2C_PH.1, LEVEL_CW.4, LEVEL_CW1.4, LEVEL_MAX.4, LEVEL_MAX1.4, LEVEL_MED.4, LEVEL_MED1.4, LEVEL_MIN.4, LEVEL_MIN1.4, R5.2, R6.2, R7.2
- net WATER: now also U$2.GPIO_69
Other:
- note added: "DHT_AM2302"
- note added: "DS18b20"
- moved on the sheet: R1, R10, R11, R12, R2, R3, R4, R5, R6, R7, R8, R9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
